File: kicad/icehat_fpga.sch (KiCad schematic (older format))
At the start: 29 parts, among them P401 CONN_02X06, P402 CONN_01X03, P403 CONN_02X06, P404 CONN_02X06, P405 CONN_01X03, P406 CONN_01X03, U401 ice5lp4k_sg48

Commit message: Fix some component values
Parts:
- R406: value 10k -> 100
Changed lines of the file:
@@
 P 9800 4350
 F 0 "R406" V 9880 4350 50  0000 C CNN
-F 1 "10k" V 9800 4350 50  0000 C CNN
+F 1 "100" V 9800 4350 50  0000 C CNN
 F 2 "Resistors_SMD:R_0603" V 9730 4350 50  0001 C CNN
 F 3 "" H 9800 4350 50  0000 C CNN
