File: kicad/icehat_pwr.sch (KiCad schematic (older format))
At the start: 6 parts, among them U301 MCP1802-3.3, U302 MCP1802-1.2

Commit message: Fix some component values
Parts:
- U302: value MCP1802-1.2 -> MCP1824-1.2
Changed lines of the file:
@@
 P 5450 4750
 F 0 "U302" H 5800 5100 60  0000 C CNN
-F 1 "MCP1802-1.2" H 5250 5100 60  0000 C CNN
+F 1 "MCP1824-1.2" H 5250 5100 60  0000 C CNN
 F 2 "TO_SOT_Packages_SMD:SOT-23-5" H 5600 4800 60  0001 C CNN
 F 3 "" H 5600 4800 60  0000 C CNN
